File: board/accel.kicad_pcb (KiCad board)
At the start: 2 copper layers, 26.7 x 49 mm, 12 parts, among them U1 NodeMCU_Amica_R2, U2 LIS2HH12

Commit message: Mark board as R2 to distinguish from previously manufactured one.
Other:
- board text added: "R2"
Changed lines of the file:
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@@
   (general
     (thickness 1.6)
-    (drawings 4)
+    (drawings 5)
     (tracks 69)
     (zones 0)
@@
       (net 10 /SPI_CS))
   )
+  (gr_text R2 (at 116.84 91.44) (layer F.Cu)
+    (effects (font (size 1.5 1.5) (thickness 0.3)))
+  )
   (gr_line (start 104.14 98.552) (end 104.14 49.53) (layer Edge.Cuts) (width 0.15))
   (gr_line (start 130.81 98.552) (end 104.14 98.552) (layer Edge.Cuts) (width 0.15))
   (gr_line (start 130.81 49.53) (end 130.81 98.552) (layer Edge.Cuts) (width 0.15))
   (gr_line (start 104.14 49.53) (end 130.81 49.53) (layer Edge.Cuts) (width 0.15))
-  (via (at 117.094 51.816) (size 0.8) (drill 0.4) (layers F.Cu B.Cu) (net 2))
-  (segment (start 114.735 51.816) (end 117.094 51.816) (width 0.25) (layer B.Cu) (net 2))
-  (via (at 125.476 51.816) (size 0.8) (drill 0.4) (layers F.Cu B.Cu) (net 2))
-  (segment (start 123.371 51.816) (end 125.476 51.816) (width 0.25) (layer B.Cu) (net 2))
-  (segment (start 120.396 55.372) (end 120.396 51.816) (width 0.25) (layer B.Cu) (net 3))
-  (segment (start 111.76 55.372) (end 111.76 51.816) (width 0.25) (layer B.Cu) (net 4))
-  (segment (start 123.371 56.347) (end 123.371 55.372) (width 0.25) (layer B.Cu) (net 5))
-  (segment (start 123.371 59.232) (end 123.371 56.347) (width 0.25) (layer B.Cu) (net 5))
-  (segment (start 127.714001 63.575001) (end 123.371 59.232) (width 0.25) (layer B.Cu) (net 5))
-  (segment (start 128.980001 63.575001) (end 127.714001 63.575001) (width 0.25) (layer B.Cu) (net 5))
-  (segment (start 125.478001 66.115001) (end 114.735 55.372) (width 0.25) (layer B.Cu) (net 6))
-  (segment (start 128.980001 66.115001) (end 125.478001 66.115001) (width 0.25) (layer B.Cu) (net 6))
-  (segment (start 124.535001 73.735001) (end 124.46 73.66) (width 0.25) (layer F.Cu) (net 7))
-  (segment (start 128.980001 73.735001) (end 124.535001 73.735001) (width 0.25) (layer F.Cu) (net 7))
   (segment (start 116.405 70.612) (end 116.405 73.406) (width 0.25) (layer F.Cu) (net 1))
   (segment (start 114.392 73.406) (end 113.285 74.513) (width 0.25) (layer F.Cu) (net 1))
@@
   (segment (start 118.361999 68.655001) (end 128.980001 68.655001) (width 0.25) (layer F.Cu) (net 1))
   (segment (start 116.405 70.612) (end 118.361999 68.655001) (width 0.25) (layer F.Cu) (net 1))
+  (via (at 117.094 51.816) (size 0.8) (drill 0.4) (layers F.Cu B.Cu) (net 2))
+  (segment (start 114.735 51.816) (end 117.094 51.816) (width 0.25) (layer B.Cu) (net 2))
+  (via (at 125.476 51.816) (size 0.8) (drill 0.4) (layers F.Cu B.Cu) (net 2))
+  (segment (start 123.371 51.816) (end 125.476 51.816) (width 0.25) (layer B.Cu) (net 2))
   (segment (start 119.38 70.612) (end 119.38 73.406) (width 0.25) (layer F.Cu) (net 2))
   (segment (start 118.608653 74.177347) (end 119.38 73.406) (width 0.25) (layer F.Cu) (net 2))
@@
   (segment (start 119.963001 71.195001) (end 119.38 70.612) (width 0.25) (layer F.Cu) (net 2))
   (segment (start 128.980001 71.195001) (end 119.963001 71.195001) (width 0.25) (layer F.Cu) (net 2))
+  (segment (start 120.396 55.372) (end 120.396 51.816) (width 0.25) (layer B.Cu) (net 3))
+  (segment (start 111.76 55.372) (end 111.76 51.816) (width 0.25) (layer B.Cu) (net 4))
+  (segment (start 123.371 56.347) (end 123.371 55.372) (width 0.25) (layer B.Cu) (net 5))
+  (segment (start 123.371 59.232) (end 123.371 56.347) (width 0.25) (layer B.Cu) (net 5))
+  (segment (start 127.714001 63.575001) (end 123.371 59.232) (width 0.25) (layer B.Cu) (net 5))
+  (segment (start 128.980001 63.575001) (end 127.714001 63.575001) (width 0.25) (layer B.Cu) (net 5))
+  (segment (start 125.478001 66.115001) (end 114.735 55.372) (width 0.25) (layer B.Cu) (net 6))
+  (segment (start 128.980001 66.115001) (end 125.478001 66.115001) (width 0.25) (layer B.Cu) (net 6))
+  (segment (start 124.535001 73.735001) (end 124.46 73.66) (width 0.25) (layer F.Cu) (net 7))
+  (segment (start 128.980001 73.735001) (end 124.535001 73.735001) (width 0.25) (layer F.Cu) (net 7))
   (via (at 109.728 73.66) (size 0.8) (drill 0.4) (layers F.Cu B.Cu) (net 7))
   (segment (start 124.46 73.66) (end 109.728 73.66) (width 0.25) (layer B.Cu) (net 7))
